File: CANable_ISO_PCB/CANable_ISO_PCB.kicad_sch (KiCad schematic)
At the start: 22 parts, among them J2 KH-RJ45-56-8P8C-D, J3 KH-RJ45-56-8P8C-D, Q1 Si2301CDS, Q2 SS8050, SW2 DSWB02LHGET, U1 STM32G431C8T6, U2 HT75xx-1-SOT89, U3 TJA1051T-3, U4 ADuM1201BR, U6 B0505S-1WR3

Commit message: Schematic pretty much done.
Could do with a tidy though...
Parts:
- removed C1: 100nF, Capacitor_SMD:C_0603_1608Metric, symbol Device:C
- removed C2: 1uF, Capacitor_SMD:C_0805_2012Metric, symbol Device:C
- removed D1: ESDA6V1BC6, Package_TO_SOT_SMD:SOT-23-6, symbol Power_Protection:ESDA6V1BC6
- removed Q1: Si2301CDS, Package_TO_SOT_SMD:SOT-23, symbol Device:Q_PMOS_GSD
- removed Q2: SS8050, Package_TO_SOT_SMD:SOT-23, symbol Transistor_BJT:BC817
- added C10, C11, C13: 1uF, Capacitor_SMD:C_0805_2012Metric, symbol Device:C
- added C12, C15, C16, C19, C23, C3, C4, C5, C6, C7, C8, C9: 100nF, Capacitor_SMD:C_0603_1608Metric, symbol Device:C
- added C14, C17, C18, C22, C24: 4.7uF, Capacitor_SMD:C_0805_2012Metric, symbol Device:C
- added D1: Red, LED_SMD:LED_0603_1608Metric, symbol Device:LED
- added D2: Blue, LED_SMD:LED_0603_1608Metric, symbol Device:LED
- added D3: Green, LED_SMD:LED_0603_1608Metric, symbol Device:LED
- added J1: USB_C_Receptacle_USB2.0, Connector_USB:USB_C_Receptacle_XKB_U262-16XN-4BVC11, symbol Connector:USB_C_Receptacle_USB2.0
- added Q1, Q2: AO3401A, Package_TO_SOT_SMD:SOT-23, symbol Transistor_FET:AO3401A
- added Q6: SS8050, Package_TO_SOT_SMD:SOT-23, symbol Transistor_BJT:BC817
- added R10, R11: 5.1k, Resistor_SMD:R_0603_1608Metric, symbol Device:R
- added R12, R13: 120R, Resistor_SMD:R_0603_1608Metric, symbol Device:R
- added R14, R15, R21, R22, R23, R25: 1k, Resistor_SMD:R_0603_1608Metric, symbol Device:R
- added R16, R6: 10k, Resistor_SMD:R_0603_1608Metric, symbol Device:R
- added R7: 1M, Resistor_SMD:R_0603_1608Metric, symbol Device:R
- added R8: 100k, Resistor_SMD:R_0603_1608Metric, symbol Device:R
- added R9: 0R, Resistor_SMD:R_0603_1608Metric, symbol Device:R
- added SW1: BOOT, Button_Switch_SMD:SW_Push_1P1T_XKB_TS-1187A, symbol Switch:SW_SPST
- added TP1, TP10, TP11, TP12, TP13, TP14, TP18, TP19, TP2, TP3, TP4, TP5, TP6, TP7, TP8, TP9: TestPoint, TestPoint:TestPoint_THTPad_1.0x1.0mm_Drill0.5mm, symbol Connector:TestPoint
- added U5, U7: TPD4E1U06DCKR, Package_TO_SOT_SMD:SOT-363_SC-70-6, symbol CANable_ISO_PCB:TPD4E1U06DCKR
- added U8: NC7SZ125P5X, Package_TO_SOT_SMD:SOT-353_SC-70-5, symbol 74xGxx:NC7SZ125P5X
- R2: value 10k -> 1k; LCSC Part # C25804 -> C21190; Manufacturer Part # 0603WAF1002T5E -> 0603WAF1001T5E
- R3: value 1k -> 100k; LCSC Part # C21190 -> C25803; Manufacturer Part # 0603WAF1001T5E -> 0603WAF1003T5E
- R5: value 5.1k -> 1k; LCSC Part # C23186 -> C21190; Manufacturer Part # 0603WAF5101T5E -> 0603WAF1001T5E
- U2: value HT75xx-1-SOT89 -> HT7533-1
Connections:
- net 0V_ISO is gone; now on net GND1: J2.11, R1.2, U3.2 (GND), U4.5 (GND2), U6.3 (-VOUT)
- net 8_way_select1/SELECTED is gone; now on net CAN_L: U3.6 (CANL)
- net +5V: now also U2.2 (VIN), C11.1, C17.1, J1.A4 (VBUS), J1.A9 (VBUS), J1.B4 (VBUS), J1.B9 (VBUS), TP5.1; no longer U4.1 (VDD1)
- net 5V_ISO: now also J2.10, J3.10, C12.1, C13.1, C14.1, C18.1, C19.1, Q1.2 (S), Q2.2 (S), R12.1, TP10.1; no longer J2.12
- net CAN_H: now also TP11.1, U7.1 (D1+)
- net CAN_L: now also TP12.1, U7.6 (D1-)
- net CAN_RX_ISO: now also Q1.1 (G), TP13.1
- net CAN_TX_ISO: now also Q2.1 (G), TP14.1
- net GND: now also R3.2, U1.19 (VSSA), U1.23 (VSS), U1.35 (VSS), U1.47 (VSS), U2.1 (GND), C10.2, C11.2, C15.2, C16.2, C17.2, C22.1, C23.2, C3.2, C4.2, C5.2, C6.2, C7.2, C8.2, C9.2, J1.A1 (GND), J1.A12 (GND), J1.B1 (GND), J1.B12 (GND), Q6.2 (E), R10.2, R11.2, R22.2, R9.2, TP19.1, U5.2 (G), U8.3 (GND)
- net CAN_RX_UB: now reaches U4.2 (VOA)
- net CAN_RX_UB: now also TP4.1, U8.2 (A)
- net CAN_TX: now reaches U4.3 (VIB)
- net CAN_TX: now also U1.46 (PB9), R16.2, TP3.1
- net +3.3V: now reaches U2.3 (VOUT)
- net +3.3V: now also U1.1 (VBAT), U1.20 (VREF+), U1.21 (VDDA), U1.24 (VDD), U1.36 (VDD), U1.48 (VDD), U4.1 (VDD1), C10.1, C15.1, C16.1, C24.1, C3.1, C4.1, C5.1, C6.1, C7.1, C8.1, D1.2 (A), D2.2 (A), D3.2 (A), R16.1, R6.1, R7.1, R8.1, SW1.2 (B), TP2.1, U8.5 (VCC)
- net at J2.9: now also R14.1
- net RJ45_SH: now reaches J2.SH
- net RJ45_SH: now also J3.SH
- net GND1: now reaches J3.11
- net GND1: now also C12.2, C13.2, C14.2, C18.2, C19.2, R13.2, R14.2, R15.2, TP18.1, TP9.1, U7.2 (G)
- net LED_1A: now reaches J3.12
- net LED_1A: now also R5.2
- net at J3.9: now also R15.1
- net at R2.1: now also Q1.3 (D)
- net LED_2A: now reaches R2.2
- net LED_2A: now also J2.12
- net CAN_RX_BOOT: now reaches R3.1
- net CAN_RX_BOOT: now also U1.45 (PB8), R25.1, SW1.1 (A)
- net at R5.1: now also Q2.3 (D)
- net LED_GREEN: now reaches U1.25 (PB11)
- net LED_GREEN: now also R21.2
- net USB_DN: now reaches U1.33 (PA11)
- net USB_DN: now also J1.A7 (D-), J1.B7 (D-), U5.4 (D2-)
- net USB_DP: now reaches U1.34 (PA12)
- net USB_DP: now also J1.A6 (D+), J1.B6 (D+), U5.3 (D2+)
- net SWDIO: now reaches U1.37 (PA13)
- net SWDIO: now also TP7.1
- net SWCLK: now reaches U1.38 (PA14)
- net SWCLK: now also TP8.1
- net LED_BLUE: now reaches U1.39 (PA15)
- net LED_BLUE: now also R23.2
- net NRST: now reaches U1.7 (PG10)
- net NRST: now also C9.1, R6.2, TP6.1
- net STBY_CTRL: now reaches U1.8 (PA0)
- net STBY_CTRL: now also TP1.1
- new net: D1.1 (K), R22.1
- new net: C22.2, Q6.1 (B), R7.2
- new net: D3.1 (K), R21.1
- new net: R25.2, U8.4 (Y)
- new net: R12.2, R13.1
- new net: D2.1 (K), R23.1
- new net CC1: J1.A5 (CC1), R10.1
- new net CC2: J1.B5 (CC2), R11.1
- new net USB_SHIELD: J1.S1 (SHIELD), R9.1
- new net ~{BUFF_OE}: C23.1, C24.2, Q6.3 (C), R8.2, U8.1 (~{OE})
- no-connect marks 2 -> 34
Other:
- note added: "3.3V MCU LDO"
- note added: "Buffer"
- note added: "Buffer Enable Delay"
- note added: "CAN data LEDs"
- note added: "FW V2 uses for standby control"
- note added: "Green"
- note added: "Indicator LEDs"
- note added: "Isolated"
- note added: "Non-isolated"
- note added: "Place close to each supply pin"
- note added: "STM32 decoupling"
- note added: "Tranciever decoupling"
- note added: "V2 sch labeled as word led?"
- note added: "Y <-- A"
- note added: "Yellow"
- note removed: "Switch with LED to indicate if active: - CAN termination - BOOT mode USB Connector Possibility to select RJ45 0V, CAN_H and CAN_L via solder jumpers or handbag links? Silent mode jumper? (Or map to IO?)"
- title: CANable ISO -> CANable V2 ISO
- moved on the sheet: H1, H2, H3, H4, R4, U1, U2

Commit message: Isolated side of layout in progress.
Parts:
- removed H3, H4: M4, MountingHole:MountingHole_4.3mm_M4, symbol Mechanical:MountingHole
Connections:
- net CAN_H: now also U7.6 (D1-); no longer U7.1 (D1+)
- net CAN_L: now also U7.1 (D1+); no longer U7.6 (D1-)
Other:
- moved on the sheet: H1, H2, TP11, TP12

Commit message: CANchovy Rev A release.
Parts:
- H1, H2: now left out of the parts list
- Q1, Q2: LCSC Part # (none) -> C15127
- U3: LCSC Part # (none) -> C38695; Manufacturer (none) -> NXP Semicon; Manufacturer Part # (none) -> TJA1051T/3/1J
Other:
- title: CANable V2 ISO -> CANchovy
Changed lines of the file:
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@@
   (paper "A3")
   (title_block
-    (title "CANable V2 ISO")
+    (title "CANchovy")
+    (date "2023-10-31")
     (rev "A")
     (company "N/A")
+    (comment 1 "MKS CANable V2 based")
   )
   (junction (at 354.33 152.4) (diameter 0) (color 0 0 0 0)
@@
   )
   (symbol (lib_id "Mechanical:MountingHole") (at 175.26 275.59 0) (unit 1)
-    (in_bom yes) (on_board yes) (dnp no) (fields_autoplaced)
+    (in_bom no) (on_board yes) (dnp no) (fields_autoplaced)
     (property "Reference" "H2" (at 177.8 274.32 0)
       (effects (font (size 1.27 1.27)) (justify left))
@@
       (effects (font (size 1.27 1.27)) (justify left) hide)
     )
+    (property "Manufacturer" "" (at 394.97 228.6 0)
+      (effects (font (size 1.27 1.27)) hide)
+    )
+    (property "Manufacturer Part #" "" (at 394.97 228.6 0)
+      (effects (font (size 1.27 1.27)) hide)
+    )
+    (property "LCSC Part #" "C15127" (at 394.97 228.6 0)
+      (effects (font (size 1.27 1.27)) hide)
+    )
     (pin "1")
     (pin "2")
@@
       (effects (font (size 1.27 1.27)) hide)
     )
+    (property "Manufacturer" "NXP Semicon" (at 250.19 133.35 0)
+      (effects (font (size 1.27 1.27)) hide)
+    )
+    (property "Manufacturer Part #" "TJA1051T/3/1J" (at 250.19 133.35 0)
+      (effects (font (size 1.27 1.27)) hide)
+    )
+    (property "LCSC Part #" "C38695" (at 250.19 133.35 0)
+      (effects (font (size 1.27 1.27)) hide)
+    )
     (pin "1")
     (pin "2")
@@
       (effects (font (size 1.27 1.27)) (justify left) hide)
     )
+    (property "Manufacturer" "" (at 359.41 228.6 0)
+      (effects (font (size 1.27 1.27)) hide)
+    )
+    (property "Manufacturer Part #" "" (at 359.41 228.6 0)
+      (effects (font (size 1.27 1.27)) hide)
+    )
+    (property "LCSC Part #" "C15127" (at 359.41 228.6 0)
+      (effects (font (size 1.27 1.27)) hide)
+    )
     (pin "1")
     (pin "2")
@@
   )
   (symbol (lib_id "Mechanical:MountingHole") (at 166.37 275.59 0) (unit 1)
-    (in_bom yes) (on_board yes) (dnp no) (fields_autoplaced)
+    (in_bom no) (on_board yes) (dnp no) (fields_autoplaced)
     (property "Reference" "H1" (at 168.91 274.32 0)
       (effects (font (size 1.27 1.27)) (justify left))
