File: CANable_ISO_PCB/CANable_ISO_PCB.kicad_pcb (KiCad board)
At the start: 2 copper layers, 14 parts, among them J2 KH-RJ45-56-8P8C-D, J3 KH-RJ45-56-8P8C-D, Q1 Si2301CDS, Q2 SS8050, U1 STM32G431C8T6, U2 HT75xx-1-SOT89, U3 TJA1051T-3, U4 ADuM1201AR, U6 B0505S-1WR3

Commit message: Schematic pretty much done.
Could do with a tidy though...
Parts:
- added C1: 100nF, Capacitor_SMD:C_0603_1608Metric, F.Cu at (94.5, 77.0)
- added C10: 1uF, Capacitor_SMD:C_0805_2012Metric, F.Cu at (32.7, 24.3)
- added C11: 1uF, Capacitor_SMD:C_0805_2012Metric, F.Cu at (32.7, 27.4)
- added C12: 100nF, Capacitor_SMD:C_0603_1608Metric, F.Cu at (94.5, 97.1)
- added C13: 1uF, Capacitor_SMD:C_0805_2012Metric, F.Cu at (90.3, 86.3)
- added C14: 4.7uF, Capacitor_SMD:C_0805_2012Metric, F.Cu at (90.3, 89.3)
- added C15: 100nF, Capacitor_SMD:C_0603_1608Metric, F.Cu at (98.6, 77.0)
- added C16: 100nF, Capacitor_SMD:C_0603_1608Metric, F.Cu at (120.0, 46.1)
- added C16: 4.7uF, Capacitor_SMD:C_0805_2012Metric, F.Cu at (90.3, 92.3)
- added C17: 4.7uF, Capacitor_SMD:C_0805_2012Metric, F.Cu at (90.3, 95.3)
- added C18: 4.7uF, Capacitor_SMD:C_0805_2012Metric, F.Cu at (90.3, 98.3)
- added C19: 100nF, Capacitor_SMD:C_0603_1608Metric, F.Cu at (98.6, 79.5)
- added C2: 1uF, Capacitor_SMD:C_0805_2012Metric, F.Cu at (90.3, 77.2)
- added C20: 100nF, Capacitor_SMD:C_0603_1608Metric, F.Cu at (98.6, 82.0)
- added C21: 22uF, Capacitor_SMD:C_1206_3216Metric, F.Cu at (103.9, 100.0)
- added C22: 4.7uF, Capacitor_SMD:C_0805_2012Metric, F.Cu at (124.3, 59.8)
- added C23: 100nF, Capacitor_SMD:C_0603_1608Metric, F.Cu at (120.0, 48.7)
- added C24: 4.7uF, Capacitor_SMD:C_0805_2012Metric, F.Cu at (124.3, 62.8)
- added C3: 100nF, Capacitor_SMD:C_0603_1608Metric, F.Cu at (141.3, 138.3)
- added C4: 100nF, Capacitor_SMD:C_0603_1608Metric, F.Cu at (141.3, 140.8)
- added C5: 100nF, Capacitor_SMD:C_0603_1608Metric, F.Cu at (141.3, 143.3)
- added C6: 100nF, Capacitor_SMD:C_0603_1608Metric, F.Cu at (141.3, 145.8)
- added C7: 100nF, Capacitor_SMD:C_0603_1608Metric, F.Cu at (141.3, 148.3)
- added C8: 100nF, Capacitor_SMD:C_0603_1608Metric, F.Cu at (141.3, 150.8)
- added C9: 100nF, Capacitor_SMD:C_0603_1608Metric, F.Cu at (118.2, 145.1)
- added D1: Red, LED_SMD:LED_0603_1608Metric, F.Cu at (108.5, 172.7)
- added D2: Blue, LED_SMD:LED_0603_1608Metric, F.Cu at (108.5, 175.2)
- added D3: Green, LED_SMD:LED_0603_1608Metric, F.Cu at (108.5, 177.8)
- added J1: USB_C_Receptacle_USB2.0, Connector_USB:USB_C_Receptacle_XKB_U262-16XN-4BVC11, F.Cu at (81.3, 38.3)
- added JP1: OPT_1, Jumper:SolderJumper-2_P1.3mm_Open_TrianglePad1.0x1.5mm, F.Cu at (50.1, 132.7)
- added JP10: OPT_2, Jumper:SolderJumper-2_P1.3mm_Open_TrianglePad1.0x1.5mm, F.Cu at (48.8, 94.8)
- added JP11: OPT_3, Jumper:SolderJumper-2_P1.3mm_Open_TrianglePad1.0x1.5mm, F.Cu at (48.8, 92.2)
- added JP12: OPT_4, Jumper:SolderJumper-2_P1.3mm_Open_TrianglePad1.0x1.5mm, F.Cu at (48.8, 89.6)
- added JP13: OPT_5, Jumper:SolderJumper-2_P1.3mm_Open_TrianglePad1.0x1.5mm, F.Cu at (45.4, 97.4)
- added JP14: OPT_5, Jumper:SolderJumper-2_P1.3mm_Open_TrianglePad1.0x1.5mm, F.Cu at (45.4, 94.8)
- added JP15: OPT_5, Jumper:SolderJumper-2_P1.3mm_Open_TrianglePad1.0x1.5mm, F.Cu at (45.4, 92.2)
- added JP16: OPT_5, Jumper:SolderJumper-2_P1.3mm_Open_TrianglePad1.0x1.5mm, F.Cu at (45.4, 89.6)
- added JP17: OPT_1, Jumper:SolderJumper-2_P1.3mm_Open_TrianglePad1.0x1.5mm, F.Cu at (48.0, 107.1)
- added JP18: OPT_2, Jumper:SolderJumper-2_P1.3mm_Open_TrianglePad1.0x1.5mm, F.Cu at (48.0, 109.7)
- added JP19: OPT_3, Jumper:SolderJumper-2_P1.3mm_Open_TrianglePad1.0x1.5mm, F.Cu at (48.0, 112.3)
- added JP2: OPT_2, Jumper:SolderJumper-2_P1.3mm_Open_TrianglePad1.0x1.5mm, F.Cu at (50.1, 130.1)
- added JP20: OPT_4, Jumper:SolderJumper-2_P1.3mm_Open_TrianglePad1.0x1.5mm, F.Cu at (48.0, 114.9)
- added JP21: OPT_5, Jumper:SolderJumper-2_P1.3mm_Open_TrianglePad1.0x1.5mm, F.Cu at (51.4, 107.1)
- added JP22: OPT_5, Jumper:SolderJumper-2_P1.3mm_Open_TrianglePad1.0x1.5mm, F.Cu at (51.4, 109.7)
- added JP23: OPT_5, Jumper:SolderJumper-2_P1.3mm_Open_TrianglePad1.0x1.5mm, F.Cu at (51.4, 112.3)
- added JP24: OPT_5, Jumper:SolderJumper-2_P1.3mm_Open_TrianglePad1.0x1.5mm, F.Cu at (51.4, 114.9)
- added JP3: OPT_3, Jumper:SolderJumper-2_P1.3mm_Open_TrianglePad1.0x1.5mm, F.Cu at (50.1, 127.5)
- added JP4: OPT_4, Jumper:SolderJumper-2_P1.3mm_Open_TrianglePad1.0x1.5mm, F.Cu at (50.1, 124.9)
- added JP5: OPT_5, Jumper:SolderJumper-2_P1.3mm_Open_TrianglePad1.0x1.5mm, F.Cu at (46.7, 132.7)
- added JP6: OPT_5, Jumper:SolderJumper-2_P1.3mm_Open_TrianglePad1.0x1.5mm, F.Cu at (46.7, 130.1)
- added JP7: OPT_5, Jumper:SolderJumper-2_P1.3mm_Open_TrianglePad1.0x1.5mm, F.Cu at (46.7, 127.5)
- added JP8: OPT_5, Jumper:SolderJumper-2_P1.3mm_Open_TrianglePad1.0x1.5mm, F.Cu at (46.7, 124.9)
- added JP9: OPT_1, Jumper:SolderJumper-2_P1.3mm_Open_TrianglePad1.0x1.5mm, F.Cu at (48.8, 97.4)
- added Q1: AO3401A, Package_TO_SOT_SMD:SOT-23, F.Cu at (124.5, 47.1)
- added Q2: AO3401A, Package_TO_SOT_SMD:SOT-23, F.Cu at (124.5, 51.6)
- added Q6: SS8050, Package_TO_SOT_SMD:SOT-23, F.Cu at (124.5, 56.0)
- added R1: 10k, Resistor_SMD:R_0603_1608Metric, F.Cu at (98.6, 84.5)
- added R10: 5.1k, Resistor_SMD:R_0603_1608Metric, F.Cu at (78.1, 26.7)
- added R11: 5.1k, Resistor_SMD:R_0603_1608Metric, F.Cu at (78.1, 29.2)
- added R12: 120R, Resistor_SMD:R_0603_1608Metric, F.Cu at (102.6, 89.5)
- added R13: 120R, Resistor_SMD:R_0603_1608Metric, F.Cu at (102.6, 92.1)
- added R14: 1k, Resistor_SMD:R_0603_1608Metric, F.Cu at (215.1, 69.9)
- added R15: 1k, Resistor_SMD:R_0603_1608Metric, F.Cu at (215.1, 72.4)
- added R16: 10k, Resistor_SMD:R_0603_1608Metric, F.Cu at (106.6, 77.0)
- added R17: 1M, Resistor_SMD:R_0603_1608Metric, F.Cu at (106.6, 79.5)
- added R18: 100k, Resistor_SMD:R_0603_1608Metric, F.Cu at (106.6, 82.0)
- added R19: 100k, Resistor_SMD:R_0603_1608Metric, F.Cu at (106.6, 84.5)
- added R2: 10k, Resistor_SMD:R_0603_1608Metric, F.Cu at (98.6, 87.0)
- added R2: 1k, Resistor_SMD:R_0603_1608Metric, F.Cu at (120.0, 51.2)
- added R21: 1k, Resistor_SMD:R_0603_1608Metric, F.Cu at (103.5, 173.2)
- added R22: 1k, Resistor_SMD:R_0603_1608Metric, F.Cu at (103.5, 175.7)
- added R23: 1k, Resistor_SMD:R_0603_1608Metric, F.Cu at (103.5, 178.2)
- added R25: 1k, Resistor_SMD:R_0603_1608Metric, F.Cu at (120.0, 63.7)
- added R3: 100k, Resistor_SMD:R_0603_1608Metric, F.Cu at (120.0, 53.7)
- added R3: 1k, Resistor_SMD:R_0603_1608Metric, F.Cu at (98.6, 89.5)
- added R4: 120R, Resistor_SMD:R_0603_1608Metric, F.Cu at (98.6, 92.1)
- added R5: 5.1k, Resistor_SMD:R_0603_1608Metric, F.Cu at (98.6, 94.6)
- added R5: 1k, Resistor_SMD:R_0603_1608Metric, F.Cu at (120.0, 56.2)
- added R6: 10k, Resistor_SMD:R_0603_1608Metric, F.Cu at (117.9, 140.5)
- added R7: 1M, Resistor_SMD:R_0603_1608Metric, F.Cu at (120.0, 58.7)
- added R7: 10k, Resistor_SMD:R_0603_1608Metric, F.Cu at (103.2, 143.0)
- added R8: 100k, Resistor_SMD:R_0603_1608Metric, F.Cu at (120.0, 61.2)
- added R8: 0R, Resistor_SMD:R_0603_1608Metric, F.Cu at (102.6, 79.5)
- added R9: 0R, Resistor_SMD:R_0603_1608Metric, F.Cu at (78.1, 24.2)
- added SW1: BOOT, Button_Switch_SMD:SW_Push_1P1T_XKB_TS-1187A, F.Cu at (131.2, 60.4)
- added SW1: BOOT, Button_Switch_SMD:SW_Push_1P1T_XKB_TS-1187A, F.Cu at (102.9, 138.6)
- added SW2: DSWB02LHGET, Button_Switch_THT:SW_DIP_SPSTx02_Slide_9.78x7.26mm_W7.62mm_P2.54mm, F.Cu at (110.5, 89.0)
- added TP1: TestPoint, TestPoint:TestPoint_THTPad_1.0x1.0mm_Drill0.5mm, F.Cu at (128.5, 46.4)
- added TP10: TestPoint, TestPoint:TestPoint_THTPad_1.0x1.0mm_Drill0.5mm, F.Cu at (134.6, 49.5)
- added TP11: TestPoint, TestPoint:TestPoint_THTPad_1.0x1.0mm_Drill0.5mm, F.Cu at (134.6, 52.5)
- added TP12: TestPoint, TestPoint:TestPoint_THTPad_1.0x1.0mm_Drill0.5mm, F.Cu at (134.6, 55.6)
- added TP13: TestPoint, TestPoint:TestPoint_THTPad_1.0x1.0mm_Drill0.5mm, F.Cu at (137.6, 46.4)
- added TP14: TestPoint, TestPoint:TestPoint_THTPad_1.0x1.0mm_Drill0.5mm, F.Cu at (137.6, 49.5)
- added TP18: TestPoint, TestPoint:TestPoint_THTPad_1.0x1.0mm_Drill0.5mm, F.Cu at (137.6, 52.5)
- added TP19: TestPoint, TestPoint:TestPoint_THTPad_1.0x1.0mm_Drill0.5mm, F.Cu at (137.6, 55.6)
- added TP2: TestPoint, TestPoint:TestPoint_THTPad_1.0x1.0mm_Drill0.5mm, F.Cu at (128.5, 49.5)
- added TP3: TestPoint, TestPoint:TestPoint_THTPad_1.0x1.0mm_Drill0.5mm, F.Cu at (128.5, 52.5)
- added TP4: TestPoint, TestPoint:TestPoint_THTPad_1.0x1.0mm_Drill0.5mm, F.Cu at (128.5, 55.6)
- added TP5: TestPoint, TestPoint:TestPoint_THTPad_1.0x1.0mm_Drill0.5mm, F.Cu at (131.5, 46.4)
- added TP6: TestPoint, TestPoint:TestPoint_THTPad_1.0x1.0mm_Drill0.5mm, F.Cu at (131.5, 49.5)
- added TP7: TestPoint, TestPoint:TestPoint_THTPad_1.0x1.0mm_Drill0.5mm, F.Cu at (131.5, 52.5)
- added TP8: TestPoint, TestPoint:TestPoint_THTPad_1.0x1.0mm_Drill0.5mm, F.Cu at (131.5, 55.6)
- added TP9: TestPoint, TestPoint:TestPoint_THTPad_1.0x1.0mm_Drill0.5mm, F.Cu at (134.6, 46.4)
- added U5: TPD4E1U06DCKR, Package_TO_SOT_SMD:SOT-363_SC-70-6, F.Cu at (84.6, 29.7)
- added U7: TPD4E1U06DCKR, Package_TO_SOT_SMD:SOT-363_SC-70-6, F.Cu at (114.8, 100.5)
- added U8: NC7SZ125P5X, Package_TO_SOT_SMD:SOT-353_SC-70-5, F.Cu at (137.6, 59.0)
- U2: value HT75xx-1-SOT89 -> HT7533-1
- U4: value ADuM1201AR -> ADuM1201BR
- moved U2 163.7 mm to (27.8, 24.7)
- moved J2 102.0 mm to (246.3, 78.4)
- moved J3 102.0 mm to (246.3, 95.5)
- moved D1 86.2 mm to (164.5, 200.1)
- moved U1 27.3 mm to (129.7, 145.0)
Connections:
- J2 pad 1: unconnected-(J2-Pad1) -> /RJ45_1
- J2 pad 10: unconnected-(J2-Pad10) -> 5V_ISO
- J2 pad 11: unconnected-(J2-Pad11) -> GND1
- J2 pad 12: unconnected-(J2-Pad12) -> /LED_2A
- J2 pad 2: unconnected-(J2-Pad2) -> /RJ45_2
- J2 pad 3: unconnected-(J2-Pad3) -> /RJ45_3
- J2 pad 4: unconnected-(J2-Pad4) -> /RJ45_4
- J2 pad 5: unconnected-(J2-Pad5) -> /RJ45_5
- J2 pad 6: unconnected-(J2-Pad6) -> /RJ45_6
- J2 pad 7: unconnected-(J2-Pad7) -> /RJ45_7
- J2 pad 8: unconnected-(J2-Pad8) -> /RJ45_8
- J2 pad 9: unconnected-(J2-Pad9) -> Net-(J2-Pad9)
- J2 pad SH: unconnected-(J2-PadSH) -> /RJ45_SH
- J3 pad 1: unconnected-(J3-Pad1) -> /RJ45_1
- J3 pad 10: unconnected-(J3-Pad10) -> 5V_ISO
- J3 pad 11: unconnected-(J3-Pad11) -> GND1
- J3 pad 12: unconnected-(J3-Pad12) -> /LED_1A
- J3 pad 2: unconnected-(J3-Pad2) -> /RJ45_2
- J3 pad 3: unconnected-(J3-Pad3) -> /RJ45_3
- J3 pad 4: unconnected-(J3-Pad4) -> /RJ45_4
- J3 pad 5: unconnected-(J3-Pad5) -> /RJ45_5
- J3 pad 6: unconnected-(J3-Pad6) -> /RJ45_6
- J3 pad 7: unconnected-(J3-Pad7) -> /RJ45_7
- J3 pad 8: unconnected-(J3-Pad8) -> /RJ45_8
- J3 pad 9: unconnected-(J3-Pad9) -> Net-(J3-Pad9)
- J3 pad SH: unconnected-(J3-PadSH) -> /RJ45_SH
- Q1 pad 1: unconnected-(Q1-G-Pad1) -> Net-(Q1-G)
- Q1 pad 2: unconnected-(Q1-S-Pad2) -> 5V_ISO
- Q1 pad 3: unconnected-(Q1-D-Pad3) -> /CAN_VIO
- Q2 pad 1: unconnected-(Q2-B-Pad1) -> Net-(Q2-B)
- Q2 pad 2: unconnected-(Q2-E-Pad2) -> 0V_ISO
- Q2 pad 3: unconnected-(Q2-C-Pad3) -> Net-(Q1-G)
- U1 pad 1: unconnected-(U1-VBAT-Pad1) -> +3.3V
- U1 pad 19: unconnected-(U1-VSSA-Pad19) -> GND
- U1 pad 20: unconnected-(U1-VREF+-Pad20) -> +3.3V
- U1 pad 21: unconnected-(U1-VDDA-Pad21) -> +3.3V
- U1 pad 23: Net-(U1-VSS-Pad23) -> GND
- U1 pad 24: unconnected-(U1-VDD-Pad24) -> +3.3V
- U1 pad 25: unconnected-(U1-PB11-Pad25) -> /LED_GREEN
- U1 pad 33: unconnected-(U1-PA11-Pad33) -> /USB_DN
- U1 pad 34: unconnected-(U1-PA12-Pad34) -> /USB_DP
- U1 pad 35: Net-(U1-VSS-Pad23) -> GND
- U1 pad 36: unconnected-(U1-VDD-Pad36) -> +3.3V
- U1 pad 37: unconnected-(U1-PA13-Pad37) -> /SWDIO
- U1 pad 38: unconnected-(U1-PA14-Pad38) -> /SWCLK
- U1 pad 39: unconnected-(U1-PA15-Pad39) -> /LED_BLUE
- U1 pad 45: unconnected-(U1-PB8-Pad45) -> /CAN_RX_BOOT
- U1 pad 46: unconnected-(U1-PB9-Pad46) -> /CAN_TX
- U1 pad 47: Net-(U1-VSS-Pad23) -> GND
- U1 pad 48: unconnected-(U1-VDD-Pad48) -> +3.3V
- U1 pad 7: unconnected-(U1-PG10-Pad7) -> /NRST
- U1 pad 8: unconnected-(U1-PA0-Pad8) -> /STBY_CTRL
- U2 pad 1: unconnected-(U2-GND-Pad1) -> GND
- U2 pad 2: unconnected-(U2-VIN-Pad2) -> +5V
- U2 pad 3: unconnected-(U2-VOUT-Pad3) -> +3.3V
- U3 pad 1: unconnected-(U3-TXD-Pad1) -> /CAN_TX_ISO
- U3 pad 2: unconnected-(U3-GND-Pad2) -> GND1
- U3 pad 3: unconnected-(U3-VCC-Pad3) -> 5V_ISO
- U3 pad 4: unconnected-(U3-RXD-Pad4) -> /CAN_RX_ISO
- U3 pad 5: unconnected-(U3-VIO-Pad5) -> 5V_ISO
- U3 pad 6: unconnected-(U3-CANL-Pad6) -> /CAN_L
- U3 pad 7: unconnected-(U3-CANH-Pad7) -> /CAN_H
- U3 pad 8: unconnected-(U3-S-Pad8) -> /SILENT_EN
- U4 pad 1: unconnected-(U4-VDD1-Pad1) -> +3.3V
- U4 pad 2: unconnected-(U4-VOA-Pad2) -> /CAN_RX_UB
- U4 pad 3: unconnected-(U4-VIB-Pad3) -> /CAN_TX
- U4 pad 4: unconnected-(U4-GND1-Pad4) -> GND
- U4 pad 5: unconnected-(U4-GND2-Pad5) -> GND1
- U4 pad 6: unconnected-(U4-VOB-Pad6) -> /CAN_TX_ISO
- U4 pad 7: unconnected-(U4-VIA-Pad7) -> /CAN_RX_ISO
- U4 pad 8: unconnected-(U4-VDD2-Pad8) -> 5V_ISO
- U6 pad 1: unconnected-(U6--VIN-Pad1) -> GND
- U6 pad 2: unconnected-(U6-+VIN-Pad2) -> +5V
- U6 pad 3: unconnected-(U6--VOUT-Pad3) -> GND1
- U6 pad 4: unconnected-(U6-+VOUT-Pad4) -> 5V_ISO
Routing:
- net GND1: track 0.00 -> 15.7 mm
- net /CAN_L: track 0.00 -> 15.7 mm
- net /CAN_H: track 0.00 -> 15.7 mm
- net /RJ45_8: track 0.00 -> 1.65 mm
- net /RJ45_7: track 0.00 -> 1.65 mm
- net /RJ45_6: track 0.00 -> 1.65 mm
- net /RJ45_5: track 0.00 -> 1.65 mm
- net /RJ45_4: track 0.00 -> 1.57 mm
- net /RJ45_1: track 0.00 -> 1.57 mm
- net /RJ45_3: track 0.00 -> 1.48 mm
- net /RJ45_2: track 0.00 -> 1.48 mm
Other:
- board text added: "0V"
- board text added: "1"
- board text added: "2"
- board text added: "3"
- board text added: "4"
- board text added: "5"
- board text added: "6"
- board text added: "7"
- board text added: "8"
- board text added: "CAN_H"
- board text added: "CAN_L"

Commit message: Isolated side of layout in progress.
Parts:
- removed C1, C20: 100nF, Capacitor_SMD:C_0603_1608Metric
- removed the C16 at (90.3, 92.3)
- removed C2: 1uF, Capacitor_SMD:C_0805_2012Metric
- removed C21: 22uF, Capacitor_SMD:C_1206_3216Metric
- removed the D1 at (164.5, 200.1)
- removed H3, H4: M4, MountingHole:MountingHole_4.3mm_M4
- removed the Q1 at (124.5, 47.1)
- removed the Q2 at (167.4, 122.8)
- removed R17: 1M, Resistor_SMD:R_0603_1608Metric
- removed R18, R19: 100k, Resistor_SMD:R_0603_1608Metric
- removed the R2 at (98.6, 87.0)
- removed the R3 at (120.0, 53.7)
- removed the R5 at (98.6, 94.6)
- removed the R7 at (120.0, 58.7)
- removed the R8 at (120.0, 61.2)
- removed the SW1 at (131.2, 60.4)
- JP1, JP10, JP11, JP12, JP13, JP14, JP15, JP16, JP17, JP18, JP19, JP2, JP20, JP21, JP22, JP23, JP24, JP3, JP4, JP5, JP6, JP7, JP8, JP9: moved to B.Cu
- Q1: value Si2301CDS -> AO3401A
- R3: value 1k -> 100k
- R7: value 10k -> 1M
- R8: value 0R -> 100k
- moved R22 162.7 mm to (42.5, 24.9)
- moved R23 162.7 mm to (42.5, 27.4)
- moved R21 162.7 mm to (42.5, 22.4)
- moved C3 160.3 mm to (30.5, 22.4)
- moved C4 160.3 mm to (30.5, 24.9)
- moved C5 160.3 mm to (30.5, 27.4)
- moved C6 160.3 mm to (30.5, 30.0)
- moved C7 160.3 mm to (30.5, 32.5)
- moved C8 160.3 mm to (30.5, 35.0)
- moved U1 142.4 mm to (50.2, 26.9)
- moved C9 138.8 mm to (30.5, 37.5)
- moved D1 137.9 mm to (39.2, 53.3)
- moved D2 137.9 mm to (39.2, 55.9)
- moved D3 137.9 mm to (39.2, 58.5)
- moved R7 136.8 mm to (38.5, 22.4)
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Connections:
- Q1 pad 1: Net-(Q1-G) -> /CAN_RX_ISO
- Q1 pad 3: /CAN_VIO -> Net-(Q1-D)
- R3 pad 1: unconnected-(R3-Pad1) -> /CAN_RX_BOOT
- R3 pad 2: unconnected-(R3-Pad2) -> GND
- R7 pad 1: /CAN_RX_BOOT -> +3.3V
- R7 pad 2: GND -> Net-(Q6-B)
- R8 pad 1: unconnected-(R8-Pad1) -> +3.3V
- R8 pad 2: unconnected-(R8-Pad2) -> /~{BUFF_OE}
- U7 pad 1: /CAN_H -> /CAN_L
- U7 pad 6: /CAN_L -> /CAN_H
Routing:
- net /RJ45_5: track 1.65 -> 105.5 mm, vias 0 -> 2
- net /RJ45_3: track 1.48 -> 98.0 mm, vias 0 -> 4
- net /RJ45_1: track 1.57 -> 95.1 mm, vias 0 -> 4
- net /RJ45_7: track 1.65 -> 89.8 mm, vias 0 -> 4
- net /RJ45_2: track 1.48 -> 87.3 mm, vias 0 -> 4
- net /RJ45_6: track 1.65 -> 78.7 mm, vias 0 -> 4
- net /RJ45_4: track 1.57 -> 78.0 mm, vias 0 -> 4
- net /RJ45_8: track 1.65 -> 75.7 mm, vias 0 -> 4
- net /CAN_H: track 15.7 -> 60.5 mm, vias 0 -> 2
- net /CAN_L: track 15.7 -> 58.5 mm, vias 0 -> 3
- net /RJ45_SH: track 0.00 -> 41.1 mm
- net /SILENT_EN: track 0.00 -> 36.6 mm, vias 0 -> 2
- net Net-(Q2-D): track 0.00 -> 35.8 mm
- net /CAN_RX_ISO: track 0.00 -> 30.5 mm, vias 0 -> 2
- net 5V_ISO: track 0.00 -> 27.3 mm, vias 0 -> 6
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- added copper zone on In2.Cu, net 5V_ISO
- added copper zone on B.Cu, net GND1
- added copper zone on F.Cu, net GND1
- added copper zone on In1.Cu, net GND1
- added copper zone on F.Cu, net Net-(R12-Pad2)
Other:
- board outline added: 75 x 50 mm
- copper layers 2 -> 4
- board text added: "SILENT"
- board text added: "TERM"

Commit message: Layout complete for now.
Parts:
- moved C23 106.2 mm to (106.0, 106.0), turned to 180 degrees
- moved C16 106.0 mm to (115.8, 93.0)
- moved R8 105.3 mm to (108.7, 103.4), turned to 90 degrees
- moved C5 101.7 mm to (109.2, 91.8), turned to 180 degrees
- moved R7 101.0 mm to (102.3, 100.7)
- moved C6 100.4 mm to (111.0, 89.9)
- moved R3 99.5 mm to (111.8, 95.2), turned to 90 degrees
- moved R16 99.1 mm to (120.6, 93.0), turned to 90 degrees
- moved R25 96.2 mm to (113.3, 95.2), turned to 90 degrees
- moved C9 94.8 mm to (111.8, 86.3), turned to -90 degrees
- moved R6 94.0 mm to (113.3, 86.3), turned to 90 degrees
- moved C17 93.9 mm to (120.3, 77.5), turned to 180 degrees
- moved C4 93.7 mm to (99.0, 88.8), turned to 90 degrees
- moved C3 93.2 mm to (105.2, 78.2), turned to 90 degrees
- moved SW1 92.7 mm to (114.3, 100.2)
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Routing:
- net +3.3V: track 3.56 -> 53.5 mm, vias 0 -> 17
- net +5V: track 0.00 -> 43.1 mm, vias 0 -> 16
- net GND: track 3.56 -> 42.4 mm, vias 0 -> 114
- net /~{BUFF_OE}: track 0.00 -> 23.8 mm
- net /LED_BLUE: track 0.00 -> 23.8 mm, vias 0 -> 2
- net /CAN_TX: track 1.84 -> 23.1 mm, vias 1 -> 2
- net /USB_SHIELD: track 0.00 -> 20.5 mm
- net /LED_GREEN: track 0.00 -> 20.3 mm, vias 0 -> 2
- net /CAN_RX_BOOT: track 0.00 -> 20.2 mm
- net /CAN_RX_UB: track 1.85 -> 21.4 mm, vias 1 -> 2
- net /USB_DP: track 0.00 -> 14.3 mm
- net /USB_DN: track 0.00 -> 13.0 mm
- net /CC1: track 0.00 -> 10.9 mm, vias 0 -> 2
- net /CC2: track 0.00 -> 9.23 mm, vias 0 -> 2
- net /NRST: track 0.00 -> 6.35 mm
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- added copper zone on In2.Cu, net +3.3V
- added copper zone on B.Cu, net +5V
- added copper zone on F.Cu, net +5V
- added copper zone on B.Cu, net GND
- added copper zone on F.Cu, net GND
- added copper zone on In1.Cu, net GND
Other:
- board text added: "3V3"
- board text added: "5V"
- board text added: "5V_ISO"
- board text added: "BOOT"
- board text added: "GND"
- board text added: "GND1"
- board text added: "SWCLK"
- board text added: "SWDIO"

Commit message: CANchovy Rev A release.
Parts:
- added G***: LOGO, LOGO, B.Cu at (108.8, 100.3)

Commit message: Corrected RJ45 footprint pinout and updated PCB to correctly label solder jumpers.
Parts:
- JP1, JP17, JP9: value OPT_1 -> OPT_8
- JP10, JP18, JP2: value OPT_2 -> OPT_7
- JP11, JP19, JP3: value OPT_3 -> OPT_6
- JP12, JP20, JP4: value OPT_4 -> OPT_5
- JP13, JP21, JP5: value OPT_5 -> OPT_4
- JP14, JP22, JP6: value OPT_5 -> OPT_3
- JP15, JP23, JP7: value OPT_5 -> OPT_2
- JP16, JP24, JP8: value OPT_5 -> OPT_1
Connections:
- JP1 pad 1: /RJ45_1 -> /RJ45_8
- JP10 pad 1: /RJ45_2 -> /RJ45_7
- JP11 pad 1: /RJ45_3 -> /RJ45_6
- JP12 pad 1: /RJ45_4 -> /RJ45_5
- JP13 pad 1: /RJ45_5 -> /RJ45_4
- JP14 pad 1: /RJ45_6 -> /RJ45_3
- JP15 pad 1: /RJ45_7 -> /RJ45_2
- JP16 pad 1: /RJ45_8 -> /RJ45_1
- JP17 pad 1: /RJ45_1 -> /RJ45_8
- JP18 pad 1: /RJ45_2 -> /RJ45_7
- JP19 pad 1: /RJ45_3 -> /RJ45_6
- JP2 pad 1: /RJ45_2 -> /RJ45_7
- JP20 pad 1: /RJ45_4 -> /RJ45_5
- JP21 pad 1: /RJ45_5 -> /RJ45_4
- JP22 pad 1: /RJ45_6 -> /RJ45_3
- JP23 pad 1: /RJ45_7 -> /RJ45_2
- JP24 pad 1: /RJ45_8 -> /RJ45_1
- JP3 pad 1: /RJ45_3 -> /RJ45_6
- JP4 pad 1: /RJ45_4 -> /RJ45_5
- JP5 pad 1: /RJ45_5 -> /RJ45_4
- JP6 pad 1: /RJ45_6 -> /RJ45_3
- JP7 pad 1: /RJ45_7 -> /RJ45_2
- JP8 pad 1: /RJ45_8 -> /RJ45_1
- JP9 pad 1: /RJ45_1 -> /RJ45_8
Routing:
- net /RJ45_5: track 108.8 -> 82.1 mm, vias 2 -> 4
- net /RJ45_4: track 82.1 -> 108.8 mm, vias 4 -> 2
- net /RJ45_8: track 78.5 -> 98.9 mm
- net /RJ45_1: track 98.9 -> 78.5 mm
- net /RJ45_6: track 82.1 -> 101.6 mm
- net /RJ45_3: track 101.6 -> 82.1 mm
- net /RJ45_7: track 92.2 -> 90.8 mm
- net /RJ45_2: track 90.8 -> 92.2 mm
