File: CANchovy_PCB/CANchovy_PCB.kicad_pcb (KiCad board)
At the start: 4 copper layers, 75 x 50 mm, 102 parts, among them J1 USB_C_Receptacle_USB2.0, J2 KH-RJ45-56-8P8C-D, J3 KH-RJ45-56-8P8C-D, Q1 AO3401A, Q2 AO3401A, Q6 SS8050, SW1 BOOT, SW2 DSWB02LHGET, U1 STM32G431C8T6, U2 HT7533-1, U3 TJA1051T-3, U4 ADuM1201BR, U5 TPD4E1U06DCKR, U6 B0505S-1WR3, U7 TPD4E1U06DCKR, U8 NC7SZ125P5X

Commit message: Revision B release.
Changes:
- Silkscreen numbering corrected for RJ45 numberings.
- RJ45 LEDs for RX/TX now ~twice the current.
Parts:
- R2, R5: value 1k -> 510R
Changed lines of the file:
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@@
   (title_block
     (title "CANchovy")
-    (date "2023-10-31")
-    (rev "A")
+    (date "2023-11-16")
+    (rev "B")
     (company "N/A")
   )
@@
     (descr "Resistor SMD 0603 (1608 Metric), square (rectangular) end terminal, IPC_7351 nominal, (Body size source: IPC-SM-782 page 72, https://www.pcb-3d.com/wordpress/wp-content/uploads/ipc-sm-782a_amendment_1_and_2.pdf), generated with kicad-footprint-generator")
     (tags "resistor")
-    (property "LCSC Part #" "C21190")
+    (property "LCSC Part #" "C23193")
     (property "Manufacturer" "UNI-ROYAL(Uniroyal Elec)")
-    (property "Manufacturer Part #" "0603WAF1001T5E")
+    (property "Manufacturer Part #" "0603WAF5100T5E")
     (property "Sheetfile" "CANchovy_PCB.kicad_sch")
     (property "Sheetname" "")
@@
         (effects (font (size 1 1) (thickness 0.15)))
     )
-    (fp_text value "1k" (at 0 1.43 90) (layer "F.Fab")
+    (fp_text value "510R" (at 0 1.43 90) (layer "F.Fab")
         (effects (font (size 1 1) (thickness 0.15)))
     )
@@
     (descr "Resistor SMD 0603 (1608 Metric), square (rectangular) end terminal, IPC_7351 nominal, (Body size source: IPC-SM-782 page 72, https://www.pcb-3d.com/wordpress/wp-content/uploads/ipc-sm-782a_amendment_1_and_2.pdf), generated with kicad-footprint-generator")
     (tags "resistor")
-    (property "LCSC Part #" "C21190")
+    (property "LCSC Part #" "C23193")
     (property "Manufacturer" "UNI-ROYAL(Uniroyal Elec)")
-    (property "Manufacturer Part #" "0603WAF1001T5E")
+    (property "Manufacturer Part #" "0603WAF5100T5E")
     (property "Sheetfile" "CANchovy_PCB.kicad_sch")
     (property "Sheetname" "")
@@
         (effects (font (size 1 1) (thickness 0.15)))
     )
-    (fp_text value "1k" (at 0 1.43 90) (layer "F.Fab")
+    (fp_text value "510R" (at 0 1.43 90) (layer "F.Fab")
         (effects (font (size 1 1) (thickness 0.15)))
     )

Commit message: Revision C & readme updates.
Parts:
- JP1, JP17, JP9: value OPT_8 -> OPT_1
- JP10, JP18, JP2: value OPT_7 -> OPT_2
- JP11, JP19, JP3: value OPT_6 -> OPT_3
- JP12, JP20, JP4: value OPT_5 -> OPT_4
- JP13, JP21, JP5: value OPT_4 -> OPT_5
- JP14, JP22, JP6: value OPT_3 -> OPT_6
- JP15, JP23, JP7: value OPT_2 -> OPT_7
- JP16, JP24, JP8: value OPT_1 -> OPT_8
Connections:
- JP1 pad 1: /RJ45_8 -> /RJ45_1
- JP10 pad 1: /RJ45_7 -> /RJ45_2
- JP11 pad 1: /RJ45_6 -> /RJ45_3
- JP12 pad 1: /RJ45_5 -> /RJ45_4
- JP13 pad 1: /RJ45_4 -> /RJ45_5
- JP14 pad 1: /RJ45_3 -> /RJ45_6
- JP15 pad 1: /RJ45_2 -> /RJ45_7
- JP16 pad 1: /RJ45_1 -> /RJ45_8
- JP17 pad 1: /RJ45_8 -> /RJ45_1
- JP18 pad 1: /RJ45_7 -> /RJ45_2
- JP19 pad 1: /RJ45_6 -> /RJ45_3
- JP2 pad 1: /RJ45_7 -> /RJ45_2
- JP20 pad 1: /RJ45_5 -> /RJ45_4
- JP21 pad 1: /RJ45_4 -> /RJ45_5
- JP22 pad 1: /RJ45_3 -> /RJ45_6
- JP23 pad 1: /RJ45_2 -> /RJ45_7
- JP24 pad 1: /RJ45_1 -> /RJ45_8
- JP3 pad 1: /RJ45_6 -> /RJ45_3
- JP4 pad 1: /RJ45_5 -> /RJ45_4
- JP5 pad 1: /RJ45_4 -> /RJ45_5
- JP6 pad 1: /RJ45_3 -> /RJ45_6
- JP7 pad 1: /RJ45_2 -> /RJ45_7
- JP8 pad 1: /RJ45_1 -> /RJ45_8
- JP9 pad 1: /RJ45_8 -> /RJ45_1
Routing:
- net /RJ45_5: track 82.1 -> 108.8 mm, vias 4 -> 2
- net /RJ45_4: track 108.8 -> 82.1 mm, vias 2 -> 4
- net /RJ45_8: track 98.9 -> 78.5 mm
- net /RJ45_1: track 78.5 -> 98.9 mm
- net /RJ45_6: track 101.6 -> 82.1 mm
- net /RJ45_3: track 82.1 -> 101.6 mm
- net GND1: track 25.6 -> 28.5 mm
- net /RJ45_7: track 90.8 -> 92.2 mm
- net /RJ45_2: track 92.2 -> 90.8 mm
